File: kicad/PicoX68Key.kicad_pcb (KiCad board)
At the start: 2 copper layers, 33.9 x 69 mm, 20 parts, among them J1 TO_X68000, Q1 2N7000, Q1 2N7002, Q2 2N7000, Q2 2N7002, Q3 2N7000, Q3 2N7002, U1 Pico

Commit message: Begin work PCB layout
Parts:
- moved Q1 0.17 mm to (69.0, 136.4)
- moved Q3 0.17 mm to (69.0, 146.4)
- moved Q3 0.12 mm to (97.5, 145.6)
Routing:
- net 3V3: track 0.00 -> 135.1 mm, vias 0 -> 1
- net VBUS: track 0.00 -> 77.1 mm
- net MS_TX_H: track 0.00 -> 37.6 mm
- net KB_TX_H: track 0.00 -> 33.0 mm, vias 0 -> 1
- net GND: track 0.00 -> 13.5 mm
- net KB_RX_H: track 41.9 -> 33.4 mm
- net KB_TX_L: track 0.00 -> 5.08 mm
- net MS_TX_L: track 0.00 -> 4.80 mm
- net KB_RX_L: track 0.00 -> 4.80 mm
Other:
- outline, holes or cut-outs redrawn
